Commit message: moveit interface and urdf update

File: boris.urdf (robot description, URDF)
Before this commit: robot boris_ros, 17 links, 16 joints
Links:
- removed link dummy_link
- removed link elbow_link
- removed link finger_link
- added link camera_link, mass 1e-5; visual box size=0.01 0.01 0.01
- added link camera_rgb_optical_frame
- added link elbow_connection_link, mass 1; collision mesh filename=package://boris_description/meshes/elbow_connection_link.STL; visual mesh filename=package://boris_description/meshes/elbow_connection_link.STL
- added link root_link
- added link wrist_connection_link, mass 1; collision mesh filename=package://boris_description/meshes/wrist_connection_link.STL; visual mesh filename=package://boris_description/meshes/wrist_connection_link.STL
- link base_link: mass None -> 1; geometry collision mesh filename=package://boris_description/meshes/base_link.STL; visual mesh filename=package://boris_description/meshes/base_link.STL
- link base_rotation_link: geometry collision mesh filename=package://boris_description/meshes/base_rotation_link.STL; visual mesh filename=package://boris_description/meshes/base_rotation_link.STL
- link gripper_left_connection_link: geometry collision mesh filename=package://boris_description/meshes/gripper_left_connection_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; visual mesh filename=package://boris_description/meshes/gripper_left_connection_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
- link gripper_left_front_link: geometry collision mesh filename=package://boris_description/meshes/gripper_left_front_link.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; visual mesh filename=package://boris_description/meshes/gripper_left_front_link.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
- link gripper_left_link: geometry collision mesh filename=package://boris_description/meshes/gripper_left_link.STL; visual mesh filename=package://boris_description/meshes/gripper_left_link.STL
- link gripper_right_connection_link: geometry collision mesh filename=package://boris_description/meshes/gripper_right_connection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; visual mesh filename=package://boris_description/meshes/gripper_right_connection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
- link gripper_right_front_link: geometry collision mesh filename=package://boris_description/meshes/gripper_right_front_link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; visual mesh filename=package://boris_description/meshes/gripper_right_front_link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
- link gripper_right_link: geometry collision mesh filename=package://boris_description/meshes/gripper_right_link.STL; visual mesh filename=package://boris_description/meshes/gripper_right_link.STL
- link hand_link: geometry collision mesh filename=package://boris_description/meshes/hand_link.STL; visual mesh filename=package://boris_description/meshes/hand_link.STL
- link lower_arm_link: geometry collision mesh filename=package://boris_description/meshes/lower_arm_link.STL; visual mesh filename=package://boris_description/meshes/lower_arm_link.STL
- link lower_support_link: geometry collision mesh filename=package://boris_description/meshes/lower_support_link.STL; visual mesh filename=package://boris_description/meshes/lower_support_link.STL
- link upper_arm_link: geometry collision mesh filename=package://boris_description/meshes/upper_arm_link.STL; visual mesh filename=package://boris_description/meshes/upper_arm_link.STL
- link upper_support_link: geometry collision mesh filename=package://boris_description/meshes/upper_support_link.STL; visual mesh filename=package://boris_description/meshes/upper_support_link.STL
- link wrist_link: geometry collision mesh filename=package://boris_description/meshes/wrist_link.STL; visual mesh filename=package://boris_description/meshes/wrist_link.STL
Joints:
- removed joint dummy_joint
- removed joint elbow_joint
- removed joint finger_joint
- added joint base_joint: type fixed, parent root_link, child base_link, origin xyz=0 0 0 rpy=0 0 0
- added joint camera_joint: type fixed, parent base_rotation_link, child camera_link, origin xyz=0 0 0.325 rpy=0 0.5 -1.57
- added joint camera_rgb_optical_joint: type fixed, parent camera_link, child camera_rgb_optical_frame, origin xyz=0 0 0 rpy=-1.57 0 -1.57
- added joint elbow_connection_joint: type revolute, parent upper_arm_link, child elbow_connection_link, origin xyz=0 0 0.17 rpy=0 0 0, axis 0 -1 0, limit lower=-0.45 upper=1.40 effort=30.0 velocity=0.7, mimic joint=upper_arm_joint multiplier=1 offset=0
- added joint wrist_connection_joint: type revolute, parent lower_arm_link, child wrist_connection_link, origin xyz=0.17 0 0 rpy=0 0 0, axis 0 -1 0, limit lower=-0.50 upper=1.20 effort=30.0 velocity=0.7, mimic joint=lower_arm_joint multiplier=1 offset=0
- joint base_rotation_joint: parent dummy_link -> base_link
- joint gripper_left_connection_joint: mimic joint=gripper_left_joint multiplier=1 offset=0 -> joint=gripper_right_joint multiplier=1 offset=0; origin xyz=0.0172 -0.00462987633392004 -0.0666094155891838 rpy=1.94880773705823 -1.5149945428384 -0.377545489148437 -> xyz=0.0665 0.00643287951573048 0.00600000000000001 rpy=0 0 0; parent finger_link -> hand_link
- joint gripper_left_front_joint: limit lower=0.00 upper=1.00 effort=30.0 velocity=0.7 -> lower=-1.00 upper=0.00 effort=30.0 velocity=0.7; mimic joint=gripper_left_joint multiplier=-1 offset=0 -> joint=gripper_right_joint multiplier=1 offset=0; origin xyz=-0.00347301637463621 0.0297982911802257 0.0069500000000001 rpy=-3.14158470285278 -6.76225140133075E-05 3.13832942623202 -> xyz=0.029999924913916 6.71204842689066E-05 0.000250000000000028 rpy=0 0 0
- joint gripper_left_joint: mimic (none) -> joint=gripper_right_joint multiplier=1 offset=0; origin xyz=0.0302 0.00480047324341529 -0.0534125028119752 rpy=-1.59151598544766 -0.113765805320385 -3.1392402140541 -> xyz=0.0535 0.0194328795157305 0.00299999999999997 rpy=0 0 0; parent finger_link -> hand_link
- joint gripper_right_connection_joint: axis 0 0 -1 -> 0 0 1; limit lower=0.00 upper=1.00 effort=30.0 velocity=0.7 -> lower=-1.00 upper=0.00 effort=30.0 velocity=0.7; mimic joint=gripper_left_joint multiplier=-1 offset=0 -> joint=gripper_right_joint multiplier=1 offset=0; origin xyz=0.0042 -0.00462987633392001 -0.0666094155891838 rpy=-1.59152382585076 -0.117029733257198 -3.1392402140541 -> xyz=0.0664999999999999 -0.00656712048426952 0.00600000000000001 rpy=0 0 0; parent finger_link -> hand_link
- joint gripper_right_front_joint: mimic joint=gripper_left_joint multiplier=1 offset=0 -> joint=gripper_right_joint multiplier=1 offset=0; origin xyz=-0.00347301637463691 0.0297982911802257 0.00695000000000001 rpy=-6.79968002564964E-05 -3.52899069022653E-06 -1.50887443585772 -> xyz=0.0299999249139151 6.71204842689031E-05 0.00025 rpy=0 0 0
- joint gripper_right_joint: axis 0 0 -1 -> 0 0 1; limit lower=0.00 upper=1.00 effort=30.0 velocity=0.7 -> lower=-1.00 upper=0.00 effort=30.0 velocity=0.7; mimic joint=gripper_left_joint multiplier=-1 offset=0 -> (none); origin xyz=-0.00879999999999999 0.00480047324341523 -0.0534125028119751 rpy=-1.59151598544766 -0.113765805320409 -3.1392402140541 -> xyz=0.0534999999999999 -0.0195671204842695 0.003 rpy=0 0 0; parent finger_link -> hand_link
- joint hand_joint: limit lower=-3.14 upper=3.14 effort=30.0 velocity=0.7 -> lower=-1.40 upper=1.40 effort=30.0 velocity=0.7; origin xyz=0 -0.0615035978826819 -0.0219899396880796 rpy=0.000163577522470927 1.57 3.14159265229103 -> xyz=0.0339425075717842 0 -0.00785697913242348 rpy=0 0 0
- joint lower_arm_joint: axis -1 0 0 -> 0 1 0; limit lower=-1.34 upper=0.49 effort=30.0 velocity=0.7 -> lower=-0.50 upper=1.20 effort=30.0 velocity=0.7; origin xyz=0 -0.063999934489265 0.030000051384737 rpy=0 0 0 -> xyz=0.0639999585758989 0 -0.030000000000005 rpy=0 0 0; parent elbow_link -> elbow_connection_link
- joint lower_support_joint: axis -1 0 0 -> 0 1 0; limit lower=-1.34 upper=0.49 effort=30.0 velocity=0.7 -> lower=-0.50 upper=1.20 effort=30.0 velocity=0.7; mimic (none) -> joint=lower_arm_joint multiplier=1 offset=0; origin xyz=0 -0.0939980623488527 -0.0339790104160389 rpy=0 0 0 -> xyz=0.0939980350675133 0 0.0339790858858603 rpy=0 0 0; parent elbow_link -> elbow_connection_link
- joint upper_arm_joint: axis 1 0 0 -> 0 1 0; limit lower=-1.92 upper=-0.15 effort=30.0 velocity=0.7 -> lower=-0.45 upper=1.40 effort=30.0 velocity=0.7; origin xyz=0.00140595251037146 0.0289658988733059 0.071 rpy=-3.14159265358979 0 3.09309252060145 -> xyz=-0.0290000000000001 0 0.062 rpy=0 0 0
- joint upper_support_joint: axis -1 0 0 -> 0 1 0; limit lower=-1.92 upper=-0.15 effort=30.0 velocity=0.7 -> lower=-0.45 upper=1.40 effort=30.0 velocity=0.7; mimic (none) -> joint=upper_arm_joint multiplier=1 offset=0; origin xyz=-0.002650339306241 -0.0349125622934152 0.041 rpy=0 0 -0.0485001329883457 -> xyz=0.035 0 0.032 rpy=0 0 0
- joint wrist_joint: axis 1 0 0 -> -1 0 0; limit lower=-1.34 upper=0.49 effort=30.0 velocity=0.7 -> lower=-1.40 upper=1.40 effort=30.0 velocity=0.7; origin xyz=0 -0.134699619920931 0.103711197048133 rpy=0 0 0 -> xyz=0.0614993382896367 0 0.0220018496935334 rpy=0 0 0; parent lower_arm_link -> wrist_connection_link
